Commit message: final commit

File: models/stair_climber/stair_climber.urdf (robot description, URDF)
Before this commit: robot stair_climber, 14 links, 13 joints
Links:
- removed link front_proximity
- removed link kinect_rod
- removed link rear_proximity
- added link bottom_camera, mass 0.027653; collision mesh filename=package://amazon_hackon/models/stair_climber/meshes/proximi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; visual mesh filename=package://amazon_hackon/models/stair_climber/meshes/proximi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
- added link box; visual mesh filename=package://amazon_hackon/models/small_box/meshes/small_box.d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
- added link kinect, mass 0.002763; collision box size=0.073000 0.276000 0.072000; visual mesh filename=package://amazon_hackon/models/stair_climber/meshes/kinect.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 scale=0.75 0.75 0.75
- added link left_belt, mass 0.87712; visual mesh filename=package://amazon_hackon/models/stair_climber/meshes/belt.STL
- added link right_belt, mass 0.87712; visual mesh filename=package://amazon_hackon/models/stair_climber/meshes/belt.STL
- link base_link: geometry visual mesh filename=package://amazon_hackon/models/stair_climber/meshes/base_li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
- link front_left_large_wheel: geometry collision mesh filename=package://amazon_hackon/models/stair_climber/meshes/large_w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 scale=1.1 1 1.1; visual mesh filename=package://amazon_hackon/models/stair_climber/meshes/large_w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
- link front_left_small_wheel: geometry collision mesh filename=package://amazon_hackon/models/stair_climber/meshes/small_w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 scale=1.1 1 1.1; visual mesh filename=package://amazon_hackon/models/stair_climber/meshes/small_w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
- link front_right_large_wheel: geometry collision mesh filename=package://amazon_hackon/models/stair_climber/meshes/large_w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 scale=1.1 1 1.1; visual mesh filename=package://amazon_hackon/models/stair_climber/meshes/large_w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
- link front_right_small_wheel: geometry collision mesh filename=package://amazon_hackon/models/stair_climber/meshes/small_w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 scale=1.1 1 1.1; visual mesh filename=package://amazon_hackon/models/stair_climber/meshes/small_w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
- link lifter: geometry collision mesh filename=package://amazon_hackon/models/stair_climber/meshes/lifter.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; visual mesh filename=package://amazon_hackon/models/stair_climber/meshes/lifter.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
- link lifter_base: geometry collision mesh filename=package://amazon_hackon/models/stair_climber/meshes/lifter_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; visual mesh filename=package://amazon_hackon/models/stair_climber/meshes/lifter_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
- link lifter_base_imu: geometry collision mesh filename=package://amazon_hackon/models/stair_climber/meshes/lifter_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; visual mesh filename=package://amazon_hackon/models/stair_climber/meshes/lifter_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
- link lifter_imu: geometry collision mesh filename=package://amazon_hackon/models/stair_climber/meshes/lifter_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; visual mesh filename=package://amazon_hackon/models/stair_climber/meshes/lifter_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
- link rear_left_small_wheel: geometry collision mesh filename=package://amazon_hackon/models/stair_climber/meshes/small_w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 scale=1.1 1 1.1; visual mesh filename=package://amazon_hackon/models/stair_climber/meshes/small_w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
- link rear_right_small_wheel: geometry collision mesh filename=package://amazon_hackon/models/stair_climber/meshes/small_w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 scale=1.1 1 1.1; visual mesh filename=package://amazon_hackon/models/stair_climber/meshes/small_w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
Joints:
- removed joint front_proximity_joint
- removed joint kinect_rod_joint
- removed joint rear_proximity_joint
- added joint bottom_camera_joint: type fixed, parent base_link, child bottom_camera, origin xyz=0.35767 0 0.09975 rpy=0 1.5708 0, axis 0 0 0
- added joint box_joint: type fixed, parent lifter, child box, origin xyz=-0.26 0 0.0713 rpy=0 0 0, axis 0 0 0
- added joint kinect_joint: type fixed, parent base_link, child kinect, origin xyz=0.36 0 0.14 rpy=0 -0 0, axis 0 0 0
- added joint left_belt_joint: type fixed, parent base_link, child left_belt, origin xyz=-0.004278 0.255 -0.008295 rpy=-1.5708 0 0, axis 0 0 0
- added joint right_belt_joint: type fixed, parent base_link, child right_belt, origin xyz=-0.004278 -0.255 -0.008295 rpy=-1.5708 0 0, axis 0 0 0
